File: flexm68k/flexm68k.sch (KiCad schematic (older format))
At the start: 4 parts, among them J1 FPC-FFC-64, U1 MC68000

Commit message: Added LOGOs in the schematics, so the PCB will have them already. Run DRC for errors. Report only three (3) overlap for silkscreen and filled zones. No problem at all.
Parts:
- added L1: GNU GPL LOGO, RetroBitLab:Symbol_GNU-GPL_SilkScreen_Small, symbol AmigaComponents:LOGO
- added L2: AMIGA LOGO, RetroBitLab:amigaLogo_BW_31x12mm, symbol AmigaComponents:LOGO
- added L3: KiCad Logo, Symbol:KiCad-Logo2_6mm_SilkScreen, symbol AmigaComponents:LOGO
- D1: footprint (none) -> LED_SMD:LED_1206_3216Metric_Pad1.42x1.75mm_HandSolder
- R1: footprint (none) -> Resistor_SMD:R_1206_3216Metric_Pad1.30x1.75mm_HandSolder
- U1: footprint dip64_800_MOT -> RetroBitLab:MC68000_REPLACEMENT
Other:
- note added: "LOGO FOR SILKSCREEN SECTION"
Changed lines of the file:
@@
 Sheet 1 1
 Title "Primary CPU Flex Connector"
-Date "2021-06-24"
-Rev "0.1"
+Date "2021-06-27"
+Rev "0.2"
 Comp "RetroBitLab"
 Comment1 ""
@@
 F 0 "U1" H 3450 4750 60  0000 C CNN
 F 1 "MC68000" H 4300 4200 60  0000 C CNN
-F 2 "dip64_800_MOT" H 5500 3140 60  0001 C CNN
+F 2 "RetroBitLab:MC68000_REPLACEMENT" H 5500 3140 60  0001 C CNN
 F 3 "" H 4300 2900 60  0000 C CNN
 	1    4300 2900
@@
 F 0 "R1" H 8200 2650 50  0000 L CNN
 F 1 "1K" H 8400 2600 50  0000 L CNN
-F 2 "" H 8350 2650 50  0001 C CNN
+F 2 "Resistor_SMD:R_1206_3216Metric_Pad1.30x1.75mm_HandSolder" H 8350 2650 50  0001 C CNN
 F 3 "~" H 8350 2650 50  0001 C CNN
 	1    8350 2650
@@
 F 0 "D1" V 8450 3100 50  0000 R CNN
 F 1 "LED_Small" V 8350 2850 50  0001 R CNN
-F 2 "" V 8350 2950 50  0001 C CNN
+F 2 "LED_SMD:LED_1206_3216Metric_Pad1.42x1.75mm_HandSolder" V 8350 2950 50  0001 C CNN
 F 3 "~" V 8350 2950 50  0001 C CNN
 	1    8350 2950
@@
 Wire Wire Line
 	1200 5100 1200 5600
+$Comp
+L AmigaComponents:LOGO L1
+U 1 1 60D88A62
+P 8700 4500
+F 0 "L1" H 8750 4600 59  0000 L CNN
+F 1 "GNU GPL LOGO" H 8750 4450 59  0000 L CNN
+F 2 "RetroBitLab:Symbol_GNU-GPL_SilkScreen_Small" H 8700 4500 59  0001 C CNN
+F 3 "" H 8700 4500 59  0001 C CNN
+	1    8700 4500
+	1    0    0    -1
+$EndComp
+$Comp
+L AmigaComponents:LOGO L3
+U 1 1 60D8ADA7
+P 8750 4900
+F 0 "L3" H 8750 5000 59  0000 L CNN
+F 1 "KiCad Logo" H 8750 4850 59  0000 L CNN
+F 2 "Symbol:KiCad-Logo2_6mm_SilkScreen" H 8750 4900 59  0001 C CNN
+F 3 "" H 8750 4900 59  0001 C CNN
+	1    8750 4900
+	1    0    0    -1
+$EndComp
+$Comp
+L AmigaComponents:LOGO L2
+U 1 1 60D8C236
+P 8700 5300
+F 0 "L2" H 8750 5400 59  0000 L CNN
+F 1 "AMIGA LOGO" H 8750 5250 59  0000 L CNN
+F 2 "RetroBitLab:amigaLogo_BW_31x12mm" H 8700 5300 59  0001 C CNN
+F 3 "" H 8700 5300 59  0001 C CNN
+	1    8700 5300
+	1    0    0    -1
+$EndComp
+Wire Notes Line
+	8500 4300 9650 4300
+Wire Notes Line
+	9650 4300 9650 5450
+Wire Notes Line
+	9650 5450 8500 5450
+Wire Notes Line
+	8500 5450 8500 4300
+Text Notes 8150 4250 0    79   ~ 16
+LOGO FOR SILKSCREEN SECTION
 $EndSCHEMATC

Commit message: Wrong footprint for CPU. Now should be corrected
Parts:
- U1: footprint RetroBitLab:MC68000_REPLACEMENT -> RetroBitLab:DIP-64_W22.86mm_Socket_LongPads_Socket
Changed lines of the file:
@@
 F 0 "U1" H 3450 4750 60  0000 C CNN
 F 1 "MC68000" H 4300 4200 60  0000 C CNN
-F 2 "RetroBitLab:MC68000_REPLACEMENT" H 5500 3140 60  0001 C CNN
+F 2 "RetroBitLab:DIP-64_W22.86mm_Socket_LongPads_Socket" H 5500 3140 60  0001 C CNN
 F 3 "" H 4300 2900 60  0000 C CNN
 	1    4300 2900

Commit message: Modified for correct footprint CPU
Parts:
- U1: footprint RetroBitLab:DIP-64_W22.86mm_Socket_LongPads_Socket -> RetroBitLab:MC68000-RELOCATOR-MALE
Changed lines of the file:
@@
 Sheet 1 1
 Title "Primary CPU Flex Connector"
-Date "2021-06-27"
-Rev "0.2"
+Date "2021-08-08"
+Rev "0.3"
 Comp "RetroBitLab"
 Comment1 ""
@@
 F 0 "U1" H 3450 4750 60  0000 C CNN
 F 1 "MC68000" H 4300 4200 60  0000 C CNN
-F 2 "RetroBitLab:DIP-64_W22.86mm_Socket_LongPads_Socket" H 5500 3140 60  0001 C CNN
+F 2 "RetroBitLab:MC68000-RELOCATOR-MALE" H 5500 3140 60  0001 C CNN
 F 3 "" H 4300 2900 60  0000 C CNN
 	1    4300 2900
